File: KiCad/LiPo-Powered_Analog _LED_Driver.kicad_pcb (KiCad board)
At the start: 2 copper layers, 100 x 70 mm, 95 parts, among them J1 Conn_01x02_Pin, J2 Conn_01x02_Pin, J3 Conn_01x02_Pin, J4 Conn_01x02_Pin, J5 Conn_01x02_Pin, Q1 2N2907A, Q10 2N2222A, Q11 2N2907A, Q14 2N2222A, Q2 2N2222A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

Commit message: Update schematic and PCB layout. Add images
Parts:
- C6, C9: footprint Capacitor_THT:C_Disc_D5.0mm_W2.5mm_P5.00mm -> Capacitor_SMD:C_0603_1608Metric_Pad1.08x0.95mm_HandSolder; moved to B.Cu
- R17: value 12K -> 56K
- R22, R25, R28, R31: footprint Resistor_SMD:R_0603_1608Metric_Pad0.98x0.95mm_HandSolder -> Resistor_THT:R_Axial_DIN0207_L6.3mm_D2.5mm_P7.62mm_Horizontal; moved to F.Cu
- R27, R29: footprint Resistor_THT:R_Axial_DIN0207_L6.3mm_D2.5mm_P7.62mm_Horizontal -> Resistor_SMD:R_0603_1608Metric_Pad0.98x0.95mm_HandSolder; moved to B.Cu
- R43: value 1K -> 470K
- moved R29 14.6 mm to (76.5, 109.2), turned to -90 degrees
- moved R26 11.8 mm to (58.2, 101.6), turned to 90 degrees
- moved R33 11.5 mm to (61.2, 88.9)
- moved R27 10.4 mm to (58.2, 98.0)
- moved R23 10.3 mm to (62.0, 104.1), turned to 0 degrees
- moved R41 10.2 mm to (93.7, 100.6)
- moved R28 8.33 mm to (87.6, 106.7), turned to 180 degrees
- moved D4 7.62 mm to (133.6, 72.1), turned to -90 degrees
- moved R25 7.34 mm to (61.5, 101.6)
- moved D8 6.99 mm to (60.7, 108.5)
- moved R31 5.00 mm to (80.0, 103.4), turned to 0 degrees
- moved R47 4.85 mm to (79.0, 94.0)
- moved C6 4.26 mm to (82.3, 109.2), turned to -90 degrees
- moved R40 4.18 mm to (87.1, 93.0)
- moved R42 4.18 mm to (90.4, 100.6)
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Connections:
- C9 pad 1: Net-(U1C--) -> Net-(U1C-+)
- Q1 pad 3: Net-(D4-A) -> Net-(D4-K)
- R40 pad 2: Net-(U1C-+) -> Net-(U1C--)
- R41 pad 1: Net-(U1C-+) -> Net-(U1C--)
- R42 pad 1: Net-(U1C-+) -> Net-(U1C--)
- R47 pad 2: Net-(U1C--) -> Net-(U1C-+)
- R7 pad 1: Net-(D4-A) -> Net-(D4-K)
- R8 pad 2: Net-(D4-A) -> Net-(D4-K)
- U2 pad 1: Net-(D4-K) -> Net-(D4-A)
Routing:
- net Net-(D4-K): track 53.2 -> 10.2 mm
- net Net-(D4-A): track 10.2 -> 52.7 mm
- net Net-(U1C-+): track 41.4 -> 17.0 mm
- net Net-(U1B-+): track 36.6 -> 12.4 mm
- net GND: track 439.0 -> 418.0 mm
- net Net-(U1C--): track 13.2 -> 30.3 mm
- net /VREF_LED: track 127.2 -> 110.9 mm
- net Net-(D8-A): track 8.55 -> 23.7 mm
- net +VSW: track 324.8 -> 311.4 mm
- net Net-(U1D-+): track 28.8 -> 15.4 mm
- net Net-(Q6-C): track 25.6 -> 14.3 mm
- net Net-(U1A--): track 34.3 -> 23.4 mm
- net Net-(R33-Pad2): track 59.4 -> 52.5 mm
- net Net-(U1B--): track 17.8 -> 11.1 mm
- net Net-(U1D--): track 11.5 -> 15.0 mm
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