File: KiCad/LiPo-Powered_Analog _LED_Driver.kicad_sch (KiCad schematic)
At the start: 95 parts, among them J1 Conn_01x02_Pin, J2 Conn_01x02_Pin, J3 Conn_01x02_Pin, J4 Conn_01x02_Pin, J5 Conn_01x02_Pin, Q1 2N2907A, Q10 2N2222A, Q11 2N2907A, Q14 2N2222A, Q2 2N2222A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

Commit message: Update schematic and PCB layout. Add images
Parts:
- C2: value 100uF -> 220uF
- C6, C9: footprint Capacitor_THT:C_Disc_D5.0mm_W2.5mm_P5.00mm -> Capacitor_SMD:C_0603_1608Metric_Pad1.08x0.95mm_HandSolder
- R17: value 12K -> 56K
- R22, R25, R28, R31: footprint Resistor_SMD:R_0603_1608Metric_Pad0.98x0.95mm_HandSolder -> Resistor_THT:R_Axial_DIN0207_L6.3mm_D2.5mm_P7.62mm_Horizontal
- R27, R29: footprint Resistor_THT:R_Axial_DIN0207_L6.3mm_D2.5mm_P7.62mm_Horizontal -> Resistor_SMD:R_0603_1608Metric_Pad0.98x0.95mm_HandSolder
- R43: value 1K -> 470K
Connections:
- net at C9.1, R47.2: now also U1.11 (+); no longer U1.10 (-)
- net at U2.1: now also D4.2 (A); no longer D4.1 (K)
- net at Q1.3 (C), R7.1, R8.2: now also D4.1 (K); no longer D4.2 (A)
- net at R40.2, R41.1, R42.1: now also U1.10 (-); no longer U1.11 (+)
Other:
- note added: "Square wave to Triangle Wave"
- moved on the sheet: C6, D4, H1, H2, H3, H4, R28, R29, R30, R31, R32, U1D
